Commit message: adding one robot teleop example

File: ROS2_WS/ros_ws/src/airobot_description/urdf/airobot.urdf.xacro (robot description, xacro)
@@ -21,5 +21,4 @@
     <xacro:property name="wheel_z" value="${wheel_radius}"/>
     <!-- ========= Frames ========= -->
-    <link name="${prefix}odom"/>
     <!-- Base (chassis) -->
     <link name="${prefix}base_link">
@@ -39,8 +38,4 @@
       </collision>
     </link>
-    <joint name="${prefix}odom_to_base" type="fixed">
-      <parent link="${prefix}odom"/>
-      <child link="${prefix}base_link"/>
-    </joint>
     <!-- ========= Left wheel ========= -->
     <link name="${prefix}left_wheel">

Commit message: tested reset service. Tracking trajectory fix needed

File: ROS2_WS/ros_ws/src/airobot_description/urdf/airobot.urdf.xacro (robot description, xacro)
@@ -42,5 +42,5 @@
       <visual>
         <!-- URDF cylinder axis is Z by default; rotate so axis becomes Y (axle) -->
-        <origin xyz="0 ${wheel_y} ${wheel_z}" rpy="1.57079632679 0 0"/>
+        <origin xyz="0 0 0" rpy="1.57079632679 0 0"/>
         <geometry>
           <cylinder radius="${wheel_radius}" length="${wheel_width}"/>
@@ -49,5 +49,5 @@
       </visual>
       <collision>
-        <origin xyz="0 ${wheel_y} ${wheel_z}" rpy="1.57079632679 0 0"/>
+        <origin xyz="0 0 0" rpy="1.57079632679 0 0"/>
         <geometry>
           <cylinder radius="${wheel_radius}" length="${wheel_width}"/>
@@ -58,5 +58,5 @@
       <parent link="${prefix}base_link"/>
       <child link="${prefix}left_wheel"/>
-      <origin xyz="0 0 0" rpy="0 0 0"/>
+      <origin xyz="0 ${wheel_y} ${wheel_z}" rpy="0 0 0"/>
       <!-- rotate about Y (axle) -->
       <axis xyz="0 1 0"/>
@@ -65,5 +65,5 @@
     <link name="${prefix}right_wheel">
       <visual>
-        <origin xyz="0 ${-wheel_y} ${wheel_z}" rpy="1.57079632679 0 0"/>
+        <origin xyz="0 0 0" rpy="1.57079632679 0 0"/>
         <geometry>
           <cylinder radius="${wheel_radius}" length="${wheel_width}"/>
@@ -72,5 +72,5 @@
       </visual>
       <collision>
-        <origin xyz="0 ${-wheel_y} ${wheel_z}" rpy="1.57079632679 0 0"/>
+        <origin xyz="0 0 0" rpy="1.57079632679 0 0"/>
         <geometry>
           <cylinder radius="${wheel_radius}" length="${wheel_width}"/>
@@ -81,5 +81,5 @@
       <parent link="${prefix}base_link"/>
       <child link="${prefix}right_wheel"/>
-      <origin xyz="0 0 0" rpy="0 0 0"/>
+      <origin xyz="0 ${-wheel_y} ${wheel_z}" rpy="0 0 0"/>
       <axis xyz="0 1 0"/>
     </joint>

Commit message: update collision field in urdf

File: ROS2_WS/ros_ws/src/airobot_description/urdf/airobot.urdf.xacro (robot description, xacro)
@@ -34,5 +34,5 @@
         <origin xyz="0 0 ${wheel_radius + base_height/2.0}" rpy="0 0 0"/>
         <geometry>
-          <box size="${base_length} ${base_width} ${base_height}"/>
+          <box size="${base_length} ${base_width+wheel_width*2.0} ${base_height}"/>
         </geometry>
       </collision>
